File: Kicad_V6/anti_furets.kicad_pcb (KiCad board)
At the start: 2 copper layers, 74.3 x 37.5 mm, 33 parts, among them J1 Jack-DC, J2 Bornier, J3 Bornier, J4 Bornier, Q1 IRF540N, Q2 TIC226, Q3 2N3905, Q4 2N3904, U1 AMS1117-5.0, U2 ATtiny85V-10PU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

Commit message: Add files via upload
Other:
- board text added: "Triac 220V 10A"
