File: Kicad_V6/anti_furets.kicad_sch (KiCad schematic)
At the start: 33 parts, among them J1 Jack-DC, J2 Bornier, J3 Bornier, J4 Bornier, Q1 IRF540N, Q2 TIC226, Q3 2N3905, Q4 2N3904, U1 AMS1117-5.0, U2 ATtiny85V-10PU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

Commit message: Add files via upload
Other:
- note added: "Cabler uniquement si on veut utiliser un spot en 220 Vac pour faire des flash lumineux"
- note added: "Texte pour save en Kicad V7"
- note added: "schémas, code arduino ATT85, pcb et dossier kicad à télécharger sur https://github.com/kotec-le-raleur/anti_furets_V2"
